File: KICAD_PCB/KICAD_PCB.kicad_pcb (KiCad board)
At the start: 2 copper layers, 38.1 x 47.8 mm, 6 parts, among them J1 RPi, J2 Protoboard, U1 TPS7A0233DBVR

Commit message: Adição do conector genérico J3
Parts:
- added J3: GENERIC_CONN, Connector_PinSocket_2.54mm:PinSocket_2x07_P2.54mm_Vertical, B.Cu at (123.8, 73.5)
- added R1: 0R, Resistor_SMD:R_0805_2012Metric, F.Cu at (123.8, 91.8)
- added R2: 0R, Resistor_SMD:R_0805_2012Metric, F.Cu at (126.5, 91.8)
Routing:
- net TXD: track 50.9 -> 118.5 mm
- net AUX: track 54.0 -> 99.6 mm
- net M0: track 55.3 -> 100.8 mm
- net M1: track 54.2 -> 93.0 mm
- net RXD: track 54.5 -> 93.3 mm
- net VCC: track 78.2 -> 96.8 mm
- net Net-(J3-Pin_14): track 0.00 -> 2.23 mm
- net Net-(J3-Pin_13): track 0.00 -> 2.23 mm
Other:
- board size 38.1 x 47.8 mm -> 44.9 x 47.8 mm
- board text added: "GND_ON"
